File: IMU+GPS Board/USB IMU Board.brd (EAGLE design)
At the start: 55 x 70 mm, 30 parts, among them J1 Adafruit GPS, Y1 16Mhz

Commit message: Version 3b
Parts:
- added C8: 100nF, SparkFun-Passives:0805
- added R2, R3: 22, SparkFun-Resistors:0805
- moved C10 1.00 mm to (29.9, 31.5), turned to 90 degrees
- moved C2 0.81 mm to (16.5, 12.0)
- moved C1 0.76 mm to (20.5, 12.4), turned to 0 degrees
- moved C5 0.50 mm to (41.1, 13.6)
- moved C6 0.22 mm to (32.7, 12.0), turned to 270 degrees
Connections:
- new net USB_N: JP1.D-, R2.1
- new net USB_P: JP1.D+, R3.1
- net DIN_N: now also R2.2; no longer JP1.D-
- net DIN_P: now also R3.2; no longer JP1.D+
- net GND: now also C8.2, U$1.33
- net VCC: now also C8.1
Routing:
- net DIN_P: track 35.2 -> 16.9 mm
- net DIN_N: track 32.4 -> 17.0 mm
- net USB_P: track 0.00 -> 15.1 mm
- net USB_N: track 0.00 -> 15.1 mm
- net VCC: track 147.3 -> 150.9 mm
- net N$1: track 7.10 -> 6.60 mm
