File: IMU+GPS Board/USB IMU Board.sch (EAGLE design)
At the start: 27 parts, among them IC1 MCP1703CB, J1 CON_HEADER_PRG_AVR_ICSP-SMD, Q1 12Mhz

Commit message: Finished with Rev.1
HW Layout done…
Parts:
- added JP2, JP3, JP4, JP5, JP6, JP7: (no value), SparkFun-Connectors:M03PTH
- added R5: 10K, SparkFun-Passives:RESISTOR0805-RES
- added R6, R7: 2.2K, SparkFun-Passives:RESISTOR0805-RES
- added U$7, U$8: FIDUCIAL, adafruit:FIDUCIAL
- C5, C6: value (none) -> 12pF
- Q1: device adafruit:CRYSTALHC49UP -> crystal_3225:CRYSTAL3.2X2.5
- Y1: value (none) -> 16 MHz
Connections:
- net DIN+ renamed DIN_P
- net DIN- renamed DIN_N
- net USB1+ renamed USB1_P
- net USB1- renamed USB1_N
- removed net 5V: JP1.VBUS, U$3.VCC, U$5.VCC, U$6.VCC
- removed net USB2+: U$3.DD+2, U$6.D+
- removed net USB2-: U$3.DD-2, U$6.D-
- removed net USB3+: U$1.D+, U$3.DD+3
- removed net USB3-: U$1.D-, U$3.DD-3
- new net 1V8: R5.2, R6.1, R7.1, U$2.VOUT
- new net GPS_RST: U$1.PB7, U$2.RST
- new net N$10: R6.2, U$2.I2C_DIO
- new net N$11: R7.2, U$2.I2C_CLK
- new net N$8: R5.1, U$2.GPIO6/CLK
- new net ON_OFF: U$2.ON_OFF, U$2.WAKEUP
- new net RX: U$1.PD3(TX), U$2.RX0/SPI_DI/HP_I2C_DIO
- new net TX: U$1.PD2(RX), U$2.TX0/SPI_DO
- new net USB2_N: U$1.D-, U$3.DD-2
- new net USB2_P: U$1.D+, U$3.DD+2
- new net USB3_N: U$3.DD-3, U$6.D-
- new net USB3_P: U$3.DD+3, U$6.D+
- net GND: now also Q1.GND, U$2.GND1, U$2.GND2, U$2.PAD
- net VCC: now also U$2.VCC_3V3
- net VUSB: now also JP1.VBUS, U$3.VCC, U$5.VCC, U$6.VCC
Other:
- note added: "Fiducials + Alignment Holes"

Commit message: Rev 0.1bc1
Fixed some things, should be ready
Parts:
- added C11, C12: (no value), SparkFun-Capacitors:CAP0805
- added LED1: GREEN, led:LEDSML0805
- added LED2: RED, led:LEDSML0805
- added R8, R9: 220, SparkFun-Resistors:RESISTOR0805-RES
- C3: value 100n -> 100nF
Connections:
- new net N$12: LED1.A, R9.1
- new net N$13: LED2.A, R8.1
- new net N$14: R9.2, U$1.PC6
- new net N$15: R8.2, U$1.PD7(ADC10)
- net GND: now also C11.2, C12.2, LED1.C, LED2.C
- net VUSB: now also C11.1, C12.1
Other:
- note added: "TODO: Power LED Status LED Decoupling Caps"
Changed lines of the file:
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@@
 <part name="R4" library="SparkFun-Passives" deviceset="RESISTOR" device="0805-RES" value="10K"/>
 <part name="GND1" library="SparkFun-Aesthetics" deviceset="GND" device=""/>
-<part name="C3" library="SparkFun-Passives" deviceset="CAP" device="0805" value="100n"/>
+<part name="C3" library="SparkFun-Passives" deviceset="CAP" device="0805" value="100nF"/>
 <part name="C4" library="SparkFun-Passives" deviceset="CAP" device="0805" value="1uF"/>
 <part name="GND2" library="SparkFun-Aesthetics" deviceset="GND" device=""/>
@@
 <part name="JP6" library="SparkFun-Connectors" deviceset="M03" device="PTH"/>
 <part name="JP7" library="SparkFun-Connectors" deviceset="M03" device="PTH"/>
+<part name="R8" library="SparkFun-Resistors" deviceset="RESISTOR" device="0805-RES" value="220"/>
+<part name="R9" library="SparkFun-Resistors" deviceset="RESISTOR" device="0805-RES" value="220"/>
+<part name="LED1" library="led" deviceset="LED" device="SML0805" value="GREEN"/>
+<part name="LED2" library="led" deviceset="LED" device="SML0805" value="RED"/>
+<part name="GND6" library="SparkFun-Aesthetics" deviceset="GND" device=""/>
+<part name="C11" library="SparkFun-Capacitors" deviceset="CAP" device="0805"/>
+<part name="C12" library="SparkFun-Capacitors" deviceset="CAP" device="0805"/>
 </parts>
 <sheets>
@@
 <instance part="C1" gate="G$1" x="114.3" y="55.88" rot="R180"/>
 <instance part="C2" gate="G$1" x="137.16" y="55.88" rot="R180"/>
+<instance part="C11" gate="G$1" x="182.88" y="50.8"/>
+<instance part="C12" gate="G$1" x="190.5" y="50.8"/>
 </instances>
 <busses>
@@
 <junction x="127" y="50.8"/>
 </segment>
+<segment>
+<pinref part="C12" gate="G$1" pin="2"/>
+<wire x1="190.5" y1="48.26" x2="182.88" y2="48.26" width="0.1524" layer="91"/>
+<label x="175.26" y="48.26" size="1.778" layer="95"/>
+<pinref part="C11" gate="G$1" pin="2"/>
+<junction x="182.88" y="48.26"/>
+<wire x1="182.88" y1="48.26" x2="177.8" y2="48.26" width="0.1524" layer="91"/>
+</segment>
 </net>
 <net name="USB1_N" class="0">
@@
 <wire x1="124.46" y1="144.78" x2="124.46" y2="154.94" width="0.1524" layer="91"/>
 <label x="124.46" y="152.4" size="1.778" layer="95" rot="R90"/>
+</segment>
+<segment>
+<pinref part="C12" gate="G$1" pin="1"/>
+<wire x1="190.5" y1="55.88" x2="182.88" y2="55.88" width="0.1524" layer="91"/>
+<label x="175.26" y="55.88" size="1.778" layer="95"/>
+<pinref part="C11" gate="G$1" pin="1"/>
+<junction x="182.88" y="55.88"/>
+<wire x1="182.88" y1="55.88" x2="177.8" y2="55.88" width="0.1524" layer="91"/>
 </segment>
 </net>
@@
 <wire x1="182.88" y1="86.36" x2="121.92" y2="86.36" width="0.254" layer="94" style="shortdash"/>
 <text x="132.08" y="50.8" size="1.778" layer="94">Fiducials + Alignment Holes</text>
+<text x="48.26" y="45.72" size="1.778" layer="91">TODO:
+Power LED
+Status LED
+Decoupling Caps</text>
 </plain>
 <instances>
@@
 <instance part="JP6" gate="G$1" x="160.02" y="60.96"/>
 <instance part="JP7" gate="G$1" x="160.02" y="76.2"/>
+<instance part="R8" gate="G$1" x="99.06" y="63.5" rot="R90"/>
+<instance part="R9" gate="G$1" x="109.22" y="63.5" rot="R90"/>
+<instance part="LED1" gate="G$1" x="109.22" y="53.34"/>
+<instance part="LED2" gate="G$1" x="99.06" y="53.34"/>
+<instance part="GND6" gate="1" x="101.6" y="43.18"/>
 </instances>
 <busses>
@@
 <label x="185.42" y="106.68" size="1.778" layer="95"/>
 </segment>
+<segment>
+<pinref part="LED2" gate="G$1" pin="C"/>
+<wire x1="99.06" y1="48.26" x2="99.06" y2="45.72" width="0.1524" layer="91"/>
+<pinref part="LED1" gate="G$1" pin="C"/>
+<wire x1="99.06" y1="45.72" x2="101.6" y2="45.72" width="0.1524" layer="91"/>
+<wire x1="101.6" y1="45.72" x2="109.22" y2="45.72" width="0.1524" layer="91"/>
+<wire x1="109.22" y1="45.72" x2="109.22" y2="48.26" width="0.1524" layer="91"/>
+<pinref part="GND6" gate="1" pin="GND"/>
+<junction x="101.6" y="45.72"/>
+</segment>
 </net>
 <net name="RST" class="0">
@@
 </segment>
 </net>
+<net name="N$12" class="0">
+<segment>
+<pinref part="R9" gate="G$1" pin="1"/>
+<pinref part="LED1" gate="G$1" pin="A"/>
+<wire x1="109.22" y1="55.88" x2="109.22" y2="58.42" width="0.1524" layer="91"/>
+</segment>
+</net>
+<net name="N$13" class="0">
+<segment>
+<pinref part="R8" gate="G$1" pin="1"/>
+<pinref part="LED2" gate="G$1" pin="A"/>
+<wire x1="99.06" y1="55.88" x2="99.06" y2="58.42" width="0.1524" layer="91"/>
+</segment>
+</net>
+<net name="N$14" class="0">
+<segment>
+<pinref part="U$1" gate="G$1" pin="PC6"/>
+<pinref part="R9" gate="G$1" pin="2"/>
+<wire x1="78.74" y1="116.84" x2="109.22" y2="116.84" width="0.1524" layer="91"/>
+<wire x1="109.22" y1="116.84" x2="109.22" y2="68.58" width="0.1524" layer="91"/>
+</segment>
+</net>
+<net name="N$15" class="0">
+<segment>
+<pinref part="U$1" gate="G$1" pin="PD7(ADC10)"/>
+<wire x1="78.74" y1="114.3" x2="106.68" y2="114.3" width="0.1524" layer="91"/>
+<wire x1="106.68" y1="114.3" x2="106.68" y2="73.66" width="0.1524" layer="91"/>
+<pinref part="R8" gate="G$1" pin="2"/>
+<wire x1="106.68" y1="73.66" x2="99.06" y2="73.66" width="0.1524" layer="91"/>
+<wire x1="99.06" y1="73.66" x2="99.06" y2="68.58" width="0.1524" layer="91"/>
+</segment>
+</net>

Commit message: Tore up USB junk
Parts:
- removed C1, C2: 20pF, SparkFun-Passives:CAP0805
- removed Q1: 12Mhz, crystal_3225:CRYSTAL3.2X2.5
- removed R1: 649, SparkFun-Passives:RESISTOR0805-RES
- removed R2: 10K, SparkFun-Passives:RESISTOR0805-RES
- removed R3: 100K, SparkFun-Passives:RESISTOR0805-RES
- removed U$3: CY7C65642, NASA Parts Lib:CY7C65642
- removed U$5, U$6: USB-SOCKET, NASA Parts Lib:USB-SOCKET
Connections:
- removed net HUB_VCC: R2.2, R3.2, U$3.SEL27, U$3.SEL48, U$3.VCC_A_1, U$3.VCC_A_12, U$3.VCC_A_16, U$3.VCC_A_19, U$3.VCC_A_7, U$3.VCC_D_34, U$3.VCC_D_38, U$3.VREG
- removed net N$1: R1.2, U$3.RREF
- removed net N$2: R3.1, U$3.GANG
- removed net N$4: C1.2, Q1.1, U$3.XIN
- removed net N$6: C2.2, Q1.2, U$3.XOUT
- removed net RESET: R2.1, U$3.RESET#
- removed net USB1_N: U$3.DD-1, U$5.D-
- removed net USB1_P: U$3.DD+1, U$5.D+
- removed net USB3_N: U$3.DD-3, U$6.D-
- removed net USB3_P: U$3.DD+3, U$6.D+
- net DIN_N: no longer U$3.DD-0
- net DIN_P: no longer U$3.DD+0
- net GND: no longer C1.1, C2.1, Q1.GND, R1.1, U$3.GND_13, U$3.GND_2, U$3.GND_20, U$3.GND_8\, U$3.SELFPWR, U$3.TEST, U$5.GND, U$5.SHLD, U$6.GND, U$6.SHLD
- net USB2_N: no longer U$3.DD-2
- net USB2_P: no longer U$3.DD+2
- net VUSB: no longer U$3.VCC, U$5.VCC, U$6.VCC
Other:
- note removed: "USB Hub Controller"
- note removed: "USB-A Jacks"

Commit message: First Round of new board
Parts:
- removed C11, C12: (no value), SparkFun-Capacitors:CAP0805
- removed JP2, JP6: (no value), SparkFun-Connectors:M03PTH
- added D1: (no value), SparkFun-DiscreteSemi:DIODESMA
- added LED3: BLUE, led:LEDSML0805
- added R1: 220, SparkFun-Resistors:RESISTOR0805-RES
- added R2: 10K, SparkFun-Resistors:RESISTOR0805-RES
- added S1: (no value), SparkFun-Electromechanical:SWITCH-SPDTPTH
- added SW1: (no value), SparkFun-Electromechanical:SWITCH_SPST_4_PIN
- added U$3: 3V, NASA Parts Lib:BU2032SM-G
- FRAME1, FRAME2: VERSION A -> 2
- Y1: value 16 MHz -> 16Mhz
Connections:
- removed net N$14: R9.2, U$1.PC6
- removed net N$15: R8.2, U$1.PD7(ADC10)
- removed net USB2_N: U$1.D-
- removed net USB2_P: U$1.D+
- new net 3V3IN: D1.C, IC1.VO, S1.P
- new net LED1: R9.2, U$1.PD7(ADC10)
- new net LED2: R8.2, U$1.PD6(ADC9)
- new net N$4: LED3.A, R1.2
- new net N$5: D1.A, U$3.PVCC
- new net PWRBTN: R2.2, SW1.1, SW1.2, U$1.PB4(ADC11)
- net DIN_N: now also U$1.D-
- net DIN_P: now also U$1.D+
- net GND: now also LED3.C, SW1.3, SW1.4, U$3.PGND; no longer C11.2, C12.2
- net VCC: now also R1.1, R2.1, S1.S; no longer IC1.VO, J1.+V
- net VUSB: now also J1.+V; no longer C11.1, C12.1
Other:
- note added: "Coin Cell / Power Switch"
- note added: "Filter Caps"
- note added: "Power Button"
- note added: "Status LEDs"
- note added: "USB (Upstream)"
- note added: "VUSB: 5.0V VCC: 3.3V"
- note removed: "TODO: Power LED Status LED Decoupling Caps"
- note removed: "Upstream USB-B Jack"

Commit message: Rev 0.2bc1 (todo: Hand Review)
Parts:
- LED1: value GREEN -> GR
- LED2: value RED -> RD
- LED3: value BLUE -> BL
- renumbered J1 to ICSP, SW1 to SHUTDOWN
Changed lines of the file:
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@@
 <?xml version="1.0" encoding="utf-8"?>
 <!DOCTYPE eagle SYSTEM "eagle.dtd">
-<eagle version="7.2.0">
+<eagle version="7.5.0">
 <drawing>
 <settings>
@@
 <part name="C9" library="SparkFun-Passives" deviceset="CAP" device="0805" value="1uF"/>
 <part name="C10" library="SparkFun-Passives" deviceset="CAP" device="0805" value="100nF"/>
-<part name="J1" library="dp_devices" deviceset="CON_HEADER_PRG_AVR_ICSP" device="-SMD"/>
+<part name="ICSP" library="dp_devices" deviceset="CON_HEADER_PRG_AVR_ICSP" device="-SMD"/>
 <part name="R5" library="SparkFun-Passives" deviceset="RESISTOR" device="0805-RES" value="10K"/>
 <part name="R6" library="SparkFun-Passives" deviceset="RESISTOR" device="0805-RES" value="2.2K"/>
@@
 <part name="R8" library="SparkFun-Resistors" deviceset="RESISTOR" device="0805-RES" value="220"/>
 <part name="R9" library="SparkFun-Resistors" deviceset="RESISTOR" device="0805-RES" value="220"/>
-<part name="LED1" library="led" deviceset="LED" device="SML0805" value="GREEN"/>
-<part name="LED2" library="led" deviceset="LED" device="SML0805" value="RED"/>
+<part name="LED1" library="led" deviceset="LED" device="SML0805" value="GR"/>
+<part name="LED2" library="led" deviceset="LED" device="SML0805" value="RD"/>
 <part name="GND6" library="SparkFun-Aesthetics" deviceset="GND" device=""/>
 <part name="U$3" library="NASA Parts Lib" deviceset="BU2032SM-G" device="" value="3V"/>
-<part name="LED3" library="led" deviceset="LED" device="SML0805" value="BLUE"/>
+<part name="LED3" library="led" deviceset="LED" device="SML0805" value="BL"/>
 <part name="R1" library="SparkFun-Resistors" deviceset="RESISTOR" device="0805-RES" value="220"/>
 <part name="GND7" library="SparkFun-Aesthetics" deviceset="GND" device=""/>
@@
 <attribute name="VERSION" value="2"/>
 </part>
-<part name="SW1" library="SparkFun-Electromechanical" deviceset="SWITCH_SPST_4_PIN" device=""/>
+<part name="SHUTDOWN" library="SparkFun-Electromechanical" deviceset="SWITCH_SPST_4_PIN" device=""/>
 <part name="R2" library="SparkFun-Resistors" deviceset="RESISTOR" device="0805-RES" value="10K"/>
 <part name="GND9" library="SparkFun-Aesthetics" deviceset="GND" device=""/>
@@
 <instance part="C7" gate="G$1" x="83.82" y="12.7"/>
 <instance part="C8" gate="G$1" x="91.44" y="12.7"/>
-<instance part="J1" gate="J" x="33.02" y="17.78"/>
+<instance part="ICSP" gate="J" x="33.02" y="17.78"/>
 <instance part="R5" gate="G$1" x="134.62" y="147.32" rot="R90"/>
 <instance part="R6" gate="G$1" x="231.14" y="149.86" rot="R90"/>
@@
 </segment>
 <segment>
-<pinref part="J1" gate="J" pin="GND"/>
+<pinref part="ICSP" gate="J" pin="GND"/>
 <wire x1="40.64" y1="15.24" x2="48.26" y2="15.24" width="0.1524" layer="91"/>
 <label x="45.72" y="15.24" size="1.778" layer="95"/>
@@
 </segment>
 <segment>
-<pinref part="J1" gate="J" pin="RST"/>
+<pinref part="ICSP" gate="J" pin="RST"/>
 <wire x1="25.4" y1="15.24" x2="17.78" y2="15.24" width="0.1524" layer="91"/>
 <label x="15.24" y="15.24" size="1.778" layer="95"/>
@@
 </segment>
 <segment>
-<pinref part="J1" gate="J" pin="+V"/>
+<pinref part="ICSP" gate="J" pin="+V"/>
 <wire x1="40.64" y1="20.32" x2="48.26" y2="20.32" width="0.1524" layer="91"/>
 <label x="45.72" y="20.32" size="1.778" layer="95"/>
@@
 <net name="MISO" class="0">
 <segment>
-<pinref part="J1" gate="J" pin="MISO"/>
+<pinref part="ICSP" gate="J" pin="MISO"/>
 <wire x1="25.4" y1="20.32" x2="17.78" y2="20.32" width="0.1524" layer="91"/>
 <label x="15.24" y="20.32" size="1.778" layer="95"/>
@@
 <net name="SCK" class="0">
 <segment>
-<pinref part="J1" gate="J" pin="SCK"/>
+<pinref part="ICSP" gate="J" pin="SCK"/>
 <wire x1="25.4" y1="17.78" x2="17.78" y2="17.78" width="0.1524" layer="91"/>
 <label x="15.24" y="17.78" size="1.778" layer="95"/>
@@
 <net name="MOSI" class="0">
 <segment>
-<pinref part="J1" gate="J" pin="MOSI"/>
+<pinref part="ICSP" gate="J" pin="MOSI"/>
 <wire x1="40.64" y1="17.78" x2="48.26" y2="17.78" width="0.1524" layer="91"/>
 <label x="45.72" y="17.78" size="1.778" layer="95"/>
@@
 <instance part="LED2" gate="G$1" x="114.3" y="162.56" rot="R90"/>
 <instance part="GND6" gate="1" x="127" y="165.1"/>
-<instance part="SW1" gate="G$1" x="177.8" y="157.48"/>
+<instance part="SHUTDOWN" gate="G$1" x="177.8" y="157.48"/>
 <instance part="R2" gate="G$1" x="167.64" y="162.56" rot="R270"/>
 <instance part="GND9" gate="1" x="193.04" y="149.86"/>
@@
 </segment>
 <segment>
-<pinref part="SW1" gate="G$1" pin="3"/>
+<pinref part="SHUTDOWN" gate="G$1" pin="3"/>
 <wire x1="182.88" y1="157.48" x2="185.42" y2="157.48" width="0.1524" layer="91"/>
 <wire x1="185.42" y1="157.48" x2="193.04" y2="157.48" width="0.1524" layer="91"/>
 <wire x1="193.04" y1="157.48" x2="193.04" y2="152.4" width="0.1524" layer="91"/>
-<pinref part="SW1" gate="G$1" pin="4"/>
+<pinref part="SHUTDOWN" gate="G$1" pin="4"/>
 <wire x1="182.88" y1="154.94" x2="185.42" y2="154.94" width="0.1524" layer="91"/>
 <wire x1="185.42" y1="154.94" x2="185.42" y2="157.48" width="0.1524" layer="91"/>
@@
 <net name="PWRBTN" class="0">
 <segment>
-<pinref part="SW1" gate="G$1" pin="1"/>
+<pinref part="SHUTDOWN" gate="G$1" pin="1"/>
 <pinref part="R2" gate="G$1" pin="2"/>
 <wire x1="167.64" y1="157.48" x2="170.18" y2="157.48" width="0.1524" layer="91"/>
@@
 <label x="152.4" y="157.48" size="1.778" layer="95"/>
 <junction x="167.64" y="157.48"/>
-<pinref part="SW1" gate="G$1" pin="2"/>
+<pinref part="SHUTDOWN" gate="G$1" pin="2"/>
 <wire x1="170.18" y1="154.94" x2="172.72" y2="154.94" width="0.1524" layer="91"/>
 <wire x1="170.18" y1="154.94" x2="170.18" y2="157.48" width="0.1524" layer="91"/>

Commit message: Late Night
Needs Check
Parts:
- removed C7: 1uF, SparkFun-Passives:CAP0805
- removed C8: 100nF, SparkFun-Passives:CAP0805
- removed D1: (no value), SparkFun-DiscreteSemi:DIODESMA
- removed IC1: MCP1703CB, linear:MCP1703CB
- removed R2: 10K, SparkFun-Resistors:RESISTOR0805-RES
- removed R5: 10K, SparkFun-Passives:RESISTOR0805-RES
- removed R6, R7: 2.2K, SparkFun-Passives:RESISTOR0805-RES
- removed S1: (no value), SparkFun-Electromechanical:SWITCH-SPDTPTH
- removed U$2: A2235-H, NASA Parts Lib:A2235-H
- removed U$3: 3V, NASA Parts Lib:BU2032SM-G
- added C1: 1uF, SparkFun-Passives:CAP0805
- added C2: 100nF, SparkFun-Passives:CAP0805
- added J1: Adafruit GPS, SparkFun-Connectors:M09
- R1, R8, R9: value 220 -> 330
- RESET: value (none) -> RST
- renumbered SHUTDOWN to RESET
Connections:
- removed net 1V8: R5.2, R6.1, R7.1, U$2.VOUT
- removed net 3V3IN: D1.C, IC1.VO, S1.P
- removed net GPS_RST: U$1.PB7, U$2.RST
- removed net N$10: R6.2, U$2.I2C_DIO
- removed net N$11: R7.2, U$2.I2C_CLK
- removed net N$5: D1.A, U$3.PVCC
- removed net N$8: R5.1, U$2.GPIO6/CLK
- removed net ON_OFF: U$2.ON_OFF, U$2.WAKEUP
- removed net PWRBTN: R2.2, RESET.1, RESET.2, U$1.PB4(ADC11)
- removed net RX: U$1.PD3(TX), U$2.RX0/SPI_DI/HP_I2C_DIO
- removed net TX: U$1.PD2(RX), U$2.TX0/SPI_DO
- removed net VUSB: C7.1, C8.1, IC1.VI, ICSP.+V, JP1.VBUS, U$1.UVCC, U$1.VBUS
- new net GPS_EN: J1.2, U$1.PF7(ADC7)
- new net MIGO: J1.5, U$1.PD2(RX)
- new net MOGI: J1.6, U$1.PD3(TX)
- net GND: now also C1.2, C2.2, J1.7; no longer C7.2, C8.2, IC1.GND, U$2.GND1, U$2.GND2, U$2.PAD, U$3.PGND
- net RST: now also RESET.1, RESET.2
- net VCC: now also C1.1, C2.1, ICSP.+V, J1.8, JP1.VBUS, U$1.UVCC, U$1.VBUS; no longer R2.1, S1.S, U$2.VCC_3V3
Other:
- note removed: "Coin Cell / Power Switch"
- note removed: "VUSB: 5.0V VCC: 3.3V"
- note removed: "Voltage Regulator"
- moved on the sheet: C10, C9, LED3, R1

Commit message: v3 Board Run
No going back now!
Parts:
- removed FRAME1: FRAME-LETTERNO_PACKAGE, SparkFun-Aesthetics:FRAME-LETTERNO_PACKAGE
Other:
- note added: "Power LED"
- note added: "Reset Button"
- note removed: "Power Button"
