File: IMU+GPS Board/USB IMU Board.sch (EAGLE design)
At the start: 29 parts, among them J1 Adafruit GPS, Y1 16Mhz

Commit message: Version 3b
Parts:
- added C8: 100nF, SparkFun-Passives:CAP0805
- added R2, R3: 22, SparkFun-Resistors:RESISTOR0805-RES
Connections:
- new net USB_N: JP1.D-, R2.1
- new net USB_P: JP1.D+, R3.1
- net DIN_N: now also R2.2; no longer JP1.D-
- net DIN_P: now also R3.2; no longer JP1.D+
- net GND: now also C8.2, U$1.PE2/!HWB
- net VCC: now also C8.1
Other:
- moved on the sheet: C1, C10, C2, C9, JP1
Changed lines of the file:
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@@
 <part name="C1" library="SparkFun-Passives" deviceset="CAP" device="0805" value="1uF"/>
 <part name="C2" library="SparkFun-Passives" deviceset="CAP" device="0805" value="100nF"/>
+<part name="C8" library="SparkFun-Passives" deviceset="CAP" device="0805" value="100nF"/>
+<part name="R2" library="SparkFun-Resistors" deviceset="RESISTOR" device="0805-RES" value="22"/>
+<part name="R3" library="SparkFun-Resistors" deviceset="RESISTOR" device="0805-RES" value="22"/>
 </parts>
 <sheets>
@@
 <wire x1="182.88" y1="106.68" x2="182.88" y2="91.44" width="0.254" layer="94" style="shortdash"/>
 <text x="152.4" y="162.56" size="1.778" layer="91">GPS</text>
-<text x="205.74" y="175.26" size="1.778" layer="94">Filter Caps</text>
+<text x="205.74" y="180.34" size="1.778" layer="94">Filter Caps</text>
 <wire x1="182.88" y1="91.44" x2="182.88" y2="35.56" width="0.254" layer="94" style="shortdash"/>
 <wire x1="116.84" y1="137.16" x2="167.64" y2="137.16" width="0.254" layer="94" style="shortdash"/>
@@
 <wire x1="177.8" y1="137.16" x2="177.8" y2="106.68" width="0.254" layer="94" style="shortdash"/>
 <text x="170.18" y="180.34" size="1.778" layer="94">Power LED</text>
-<text x="109.22" y="27.94" size="1.778" layer="94">USB (Upstream)</text>
+<text x="73.66" y="27.94" size="1.778" layer="94">USB (Upstream)</text>
 <text x="187.96" y="119.38" size="1.778" layer="94">Reset Button</text>
 <wire x1="182.88" y1="91.44" x2="248.92" y2="91.44" width="0.254" layer="94" style="shortdash"/>
@@
 <instance part="JP7" gate="G$1" x="165.1" y="78.74"/>
 <instance part="J1" gate="G$1" x="147.32" y="162.56" rot="R180"/>
-<instance part="C9" gate="G$1" x="218.44" y="162.56"/>
-<instance part="C10" gate="G$1" x="231.14" y="162.56"/>
-<instance part="C1" gate="G$1" x="218.44" y="137.16"/>
-<instance part="C2" gate="G$1" x="231.14" y="137.16"/>
+<instance part="C9" gate="G$1" x="218.44" y="167.64"/>
+<instance part="C10" gate="G$1" x="231.14" y="167.64"/>
+<instance part="C1" gate="G$1" x="218.44" y="134.62"/>
+<instance part="C2" gate="G$1" x="231.14" y="134.62"/>
 <instance part="LED3" gate="G$1" x="182.88" y="152.4"/>
 <instance part="R1" gate="G$1" x="182.88" y="162.56" rot="R270"/>
@@
 <instance part="LED2" gate="G$1" x="152.4" y="116.84" rot="R90"/>
 <instance part="GND6" gate="1" x="165.1" y="119.38"/>
-<instance part="JP1" gate="G$1" x="121.92" y="20.32" rot="R180"/>
+<instance part="JP1" gate="G$1" x="86.36" y="20.32" rot="R180"/>
 <instance part="RESET" gate="G$1" x="215.9" y="111.76"/>
 <instance part="GND9" gate="1" x="231.14" y="104.14"/>
+<instance part="C8" gate="G$1" x="231.14" y="152.4"/>
+<instance part="R2" gate="G$1" x="111.76" y="15.24"/>
+<instance part="R3" gate="G$1" x="111.76" y="12.7"/>
 </instances>
 <busses>
@@
 <segment>
 <pinref part="C10" gate="G$1" pin="1"/>
-<wire x1="231.14" y1="170.18" x2="231.14" y2="167.64" width="0.1524" layer="91"/>
-<wire x1="231.14" y1="170.18" x2="218.44" y2="170.18" width="0.1524" layer="91"/>
+<wire x1="231.14" y1="175.26" x2="231.14" y2="172.72" width="0.1524" layer="91"/>
+<wire x1="231.14" y1="175.26" x2="218.44" y2="175.26" width="0.1524" layer="91"/>
 <pinref part="C9" gate="G$1" pin="1"/>
-<wire x1="218.44" y1="170.18" x2="210.82" y2="170.18" width="0.1524" layer="91"/>
-<wire x1="218.44" y1="167.64" x2="218.44" y2="170.18" width="0.1524" layer="91"/>
-<junction x="218.44" y="170.18"/>
-<label x="210.82" y="170.18" size="1.778" layer="95"/>
+<wire x1="218.44" y1="175.26" x2="210.82" y2="175.26" width="0.1524" layer="91"/>
+<wire x1="218.44" y1="172.72" x2="218.44" y2="175.26" width="0.1524" layer="91"/>
+<junction x="218.44" y="175.26"/>
+<label x="210.82" y="175.26" size="1.778" layer="95"/>
 </segment>
 <segment>
 <pinref part="C2" gate="G$1" pin="1"/>
-<wire x1="231.14" y1="144.78" x2="231.14" y2="142.24" width="0.1524" layer="91"/>
-<wire x1="231.14" y1="144.78" x2="218.44" y2="144.78" width="0.1524" layer="91"/>
+<wire x1="231.14" y1="142.24" x2="231.14" y2="139.7" width="0.1524" layer="91"/>
+<wire x1="231.14" y1="142.24" x2="218.44" y2="142.24" width="0.1524" layer="91"/>
 <pinref part="C1" gate="G$1" pin="1"/>
-<wire x1="218.44" y1="144.78" x2="210.82" y2="144.78" width="0.1524" layer="91"/>
-<wire x1="218.44" y1="142.24" x2="218.44" y2="144.78" width="0.1524" layer="91"/>
-<junction x="218.44" y="144.78"/>
-<label x="210.82" y="144.78" size="1.778" layer="95"/>
+<wire x1="218.44" y1="142.24" x2="210.82" y2="142.24" width="0.1524" layer="91"/>
+<wire x1="218.44" y1="139.7" x2="218.44" y2="142.24" width="0.1524" layer="91"/>
+<junction x="218.44" y="142.24"/>
+<label x="210.82" y="142.24" size="1.778" layer="95"/>
 </segment>
 <segment>
@@
 <segment>
 <pinref part="JP1" gate="G$1" pin="VBUS"/>
-<wire x1="124.46" y1="17.78" x2="134.62" y2="17.78" width="0.1524" layer="91"/>
-<label x="132.08" y="17.78" size="1.778" layer="95"/>
+<wire x1="88.9" y1="17.78" x2="99.06" y2="17.78" width="0.1524" layer="91"/>
+<label x="96.52" y="17.78" size="1.778" layer="95"/>
+</segment>
+<segment>
+<pinref part="C8" gate="G$1" pin="1"/>
+<wire x1="231.14" y1="157.48" x2="210.82" y2="157.48" width="0.1524" layer="91"/>
+<label x="210.82" y="157.48" size="1.778" layer="95"/>
 </segment>
 </net>
@@
 <wire x1="40.64" y1="76.2" x2="40.64" y2="73.66" width="0.1524" layer="91"/>
 <junction x="40.64" y="73.66"/>
+<pinref part="U$1" gate="G$1" pin="PE2/!HWB"/>
+<wire x1="48.26" y1="83.82" x2="40.64" y2="83.82" width="0.1524" layer="91"/>
+<wire x1="40.64" y1="83.82" x2="40.64" y2="76.2" width="0.1524" layer="91"/>
+<junction x="40.64" y="76.2"/>
 </segment>
 <segment>
@@
 <segment>
 <pinref part="C10" gate="G$1" pin="2"/>
-<wire x1="231.14" y1="157.48" x2="231.14" y2="160.02" width="0.1524" layer="91"/>
-<wire x1="231.14" y1="157.48" x2="218.44" y2="157.48" width="0.1524" layer="91"/>
+<wire x1="231.14" y1="165.1" x2="218.44" y2="165.1" width="0.1524" layer="91"/>
 <pinref part="C9" gate="G$1" pin="2"/>
-<wire x1="218.44" y1="157.48" x2="210.82" y2="157.48" width="0.1524" layer="91"/>
-<wire x1="218.44" y1="160.02" x2="218.44" y2="157.48" width="0.1524" layer="91"/>
-<junction x="218.44" y="157.48"/>
-<label x="210.82" y="157.48" size="1.778" layer="95"/>
+<wire x1="218.44" y1="165.1" x2="210.82" y2="165.1" width="0.1524" layer="91"/>
+<junction x="218.44" y="165.1"/>
+<label x="210.82" y="165.1" size="1.778" layer="95"/>
 </segment>
 <segment>
 <pinref part="C2" gate="G$1" pin="2"/>
-<wire x1="231.14" y1="132.08" x2="231.14" y2="134.62" width="0.1524" layer="91"/>
-<wire x1="231.14" y1="132.08" x2="218.44" y2="132.08" width="0.1524" layer="91"/>
+<wire x1="231.14" y1="129.54" x2="231.14" y2="132.08" width="0.1524" layer="91"/>
+<wire x1="231.14" y1="129.54" x2="218.44" y2="129.54" width="0.1524" layer="91"/>
 <pinref part="C1" gate="G$1" pin="2"/>
-<wire x1="218.44" y1="132.08" x2="210.82" y2="132.08" width="0.1524" layer="91"/>
-<wire x1="218.44" y1="134.62" x2="218.44" y2="132.08" width="0.1524" layer="91"/>
-<junction x="218.44" y="132.08"/>
-<label x="210.82" y="132.08" size="1.778" layer="95"/>
+<wire x1="218.44" y1="129.54" x2="210.82" y2="129.54" width="0.1524" layer="91"/>
+<wire x1="218.44" y1="132.08" x2="218.44" y2="129.54" width="0.1524" layer="91"/>
+<junction x="218.44" y="129.54"/>
+<label x="210.82" y="129.54" size="1.778" layer="95"/>
 </segment>
 <segment>
@@
 <segment>
 <pinref part="JP1" gate="G$1" pin="GND"/>
-<wire x1="124.46" y1="20.32" x2="134.62" y2="20.32" width="0.1524" layer="91"/>
-<label x="132.08" y="20.32" size="1.778" layer="95"/>
+<wire x1="88.9" y1="20.32" x2="99.06" y2="20.32" width="0.1524" layer="91"/>
+<label x="96.52" y="20.32" size="1.778" layer="95"/>
 </segment>
 <segment>
@@
 <junction x="223.52" y="111.76"/>
 </segment>
+<segment>
+<pinref part="C8" gate="G$1" pin="2"/>
+<wire x1="231.14" y1="149.86" x2="210.82" y2="149.86" width="0.1524" layer="91"/>
+<label x="210.82" y="149.86" size="1.778" layer="95"/>
+</segment>
 </net>
 <net name="RST" class="0">
@@
 </segment>
 <segment>
-<pinref part="JP1" gate="G$1" pin="D-"/>
-<wire x1="124.46" y1="15.24" x2="134.62" y2="15.24" width="0.1524" layer="91"/>
-<label x="132.08" y="15.24" size="1.778" layer="95"/>
+<pinref part="R2" gate="G$1" pin="2"/>
+<wire x1="116.84" y1="15.24" x2="124.46" y2="15.24" width="0.1524" layer="91"/>
+<label x="121.92" y="15.24" size="1.778" layer="95"/>
 </segment>
 </net>
@@
 </segment>
 <segment>
-<pinref part="JP1" gate="G$1" pin="D+"/>
-<wire x1="124.46" y1="12.7" x2="134.62" y2="12.7" width="0.1524" layer="91"/>
-<label x="132.08" y="12.7" size="1.778" layer="95"/>
+<pinref part="R3" gate="G$1" pin="2"/>
+<wire x1="116.84" y1="12.7" x2="124.46" y2="12.7" width="0.1524" layer="91"/>
+<label x="121.92" y="12.7" size="1.778" layer="95"/>
 </segment>
 </net>
@@
 </segment>
 </net>
+<net name="USB_N" class="0">
+<segment>
+<pinref part="R2" gate="G$1" pin="1"/>
+<pinref part="JP1" gate="G$1" pin="D-"/>
+<wire x1="106.68" y1="15.24" x2="88.9" y2="15.24" width="0.1524" layer="91"/>
+<label x="99.06" y="15.24" size="1.778" layer="95"/>
+</segment>
+</net>
+<net name="USB_P" class="0">
+<segment>
+<pinref part="JP1" gate="G$1" pin="D+"/>
+<pinref part="R3" gate="G$1" pin="1"/>
+<wire x1="88.9" y1="12.7" x2="106.68" y2="12.7" width="0.1524" layer="91"/>
+<label x="99.06" y="12.7" size="1.778" layer="95"/>
+</segment>
+</net>
